File: askew-kbd/askew-kbd.kicad_pcb (KiCad board)
At the start: 2 copper layers, 155.6 x 108.4 mm, 68 parts, among them J1 OLED, J2 MJ-4PP-9, SW1 SW_PUSH, SW10 SW_PUSH, SW11 SW_PUSH, SW12 SW_PUSH, SW13 SW_PUSH, SW14 SW_PUSH, SW15 SW_PUSH, SW16 SW_PUSH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

Commit message: choc_spacing
Parts:
- removed J1: OLED, kbd:OLED_v2
- removed J2: MJ-4PP-9, kbd:MJ-4PP-9
- removed JP1, JP2, JP3, JP4, JP5, JP6, JP7, JP8: , kbd:Jumper
- removed JP9: , kbd:JPC2
- removed REF** (x9): M2_Hole_TH_Outside, kbd:M2_Hole_TH_Outside
- removed REF** (x2): M2_Hole_TH, kbd:M2_Hole_TH
- removed RSW1: SW_PUSH, kbd:ResetSW
- removed U1: ProMicro, keyboard_reversible:ProMicro_unrouted
- SW1, SW10, SW11, SW12, SW13, SW14, SW15, SW16, SW17, SW18, SW2, SW21, SW3, SW4, SW5, SW6, SW7, SW8, SW9: footprint fp:ChocV1_V2_Hotswap_reversed -> fp:ChocV1_V2_Hotswap_reversed_choc_spacing
- SW19, SW20, SW22: footprint fp:ChocV1_V2_Hotswap_reversed_15u -> fp:ChocV1_V2_Hotswap_reversed_15u_choc_spacing
- moved D14 10.3 mm to (154.6, 79.1)
- moved SW7 9.53 mm to (122.8, 71.4), turned to 3 degrees
- moved D15 9.36 mm to (148.1, 116.0)
- moved SW10 9.02 mm to (143.2, 70.0)
- moved SW8 7.71 mm to (123.8, 88.5), turned to 3 degrees
- moved SW11 7.23 mm to (143.3, 87.2)
- moved SW1 7.18 mm to (79.5, 83.7)
- moved SW22 6.57 mm to (196.1, 135.8), turned to -120 degrees
- moved SW4 6.56 mm to (97.0, 79.0)
- moved D2 6.16 mm to (76.6, 99.5)
- moved D3 6.16 mm to (81.5, 117.8)
- moved D1 6.16 mm to (71.7, 81.1)
- moved SW9 5.91 mm to (124.7, 105.5), turned to 3 degrees
- moved SW2 5.87 mm to (83.9, 100.3)
- moved SW12 5.50 mm to (143.2, 104.3)
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Routing:
- net GND: track 0.52 -> 0.00 mm
Other:
- board outline removed

Commit message: redo layout
Parts:
- added J1: OLED, kbd:OLED_v2, F.Cu at (200.4, 101.5)
- added J2: MJ-4PP-9, kbd:MJ-4PP-9, F.Cu at (210.0, 108.5)
- added JP1: , kbd:Jumper, F.Cu at (258.2, 126.8)
- added JP2: , kbd:Jumper, F.Cu at (273.0, 111.6)
- added JP3: , kbd:Jumper, F.Cu at (261.6, 126.8)
- added JP4: , kbd:Jumper, F.Cu at (278.7, 126.8)
- added JP5: , kbd:Jumper, F.Cu at (275.3, 126.8)
- added JP6: , kbd:Jumper, F.Cu at (268.4, 126.8)
- added JP7: , kbd:Jumper, F.Cu at (265.7, 67.9)
- added JP8: , kbd:Jumper, F.Cu at (265.0, 126.8)
- added JP9: , kbd:JPC2, F.Cu at (271.9, 126.8)
- added RSW1: SW_PUSH, kbd:ResetSW, F.Cu at (191.9, 100.0)
- added U1: ProMicro, keyboard_reversible:ProMicro_unrouted, F.Cu at (201.5, 80.0)
- D1, D10, D11, D12, D13, D14, D15, D16, D17, D18, D19, D2, D20, D21, D22, D3, D4, D5, D6, D7, D8, D9: footprint fp:D3_SMD -> kbd:D3_TH_SMD
- moved D1 192.3 mm to (262.1, 108.4), turned to 0 degrees
- moved D3 176.5 mm to (258.1, 119.4), turned to 0 degrees
- moved D4 175.3 mm to (258.0, 123.6), turned to 0 degrees
- moved D6 171.2 mm to (269.3, 95.0), turned to 0 degrees
- moved D2 169.2 mm to (244.1, 75.3), turned to 0 degrees
- moved D5 161.9 mm to (254.8, 75.3), turned to 0 degrees
- moved D19 151.6 mm to (262.1, 115.5), turned to 0 degrees
- moved D7 150.0 mm to (253.2, 122.6), turned to 0 degrees
- moved D20 136.6 mm to (279.6, 121.3), turned to 0 degrees
- moved D8 129.5 mm to (244.1, 68.2), turned to 0 degrees
- moved D12 126.9 mm to (262.1, 112.0), turned to 0 degrees
- moved D9 125.9 mm to (242.8, 109.0), turned to 0 degrees
- moved D10 115.3 mm to (242.8, 105.5), turned to 0 degrees
- moved D11 108.3 mm to (242.8, 98.3), turned to 0 degrees
- moved D21 105.3 mm to (254.8, 68.2), turned to 0 degrees
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Routing:
- removed copper zone on F.Cu, net GND
Other:
- board outline added: 145.2 x 92.1 mm

Commit message: pro micro and diodes
Parts:
- JP5, JP6, JP7, JP8: moved to B.Cu
- U1: footprint keyboard_reversible:ProMicro_unrouted -> fp:ProMicro_unrouted_type_c
- moved D1 175.9 mm to (88.9, 77.4), turned to 105 degrees
- moved D3 162.5 mm to (95.8, 109.6), turned to 105 degrees
- moved D4 158.1 mm to (108.0, 73.8), turned to 103 degrees
- moved D6 157.0 mm to (112.7, 105.1), turned to 103 degrees
- moved D2 154.0 mm to (91.0, 92.1), turned to 105 degrees
- moved D7 149.8 mm to (112.0, 72.8), turned to 93 degrees
- moved D5 144.9 mm to (110.5, 88.3), turned to 103 degrees
- moved D8 131.7 mm to (113.3, 83.8), turned to 93 degrees
- moved D12 128.9 mm to (133.8, 99.8), turned to 90 degrees
- moved D19 128.5 mm to (133.9, 124.3), turned to 95 degrees
- moved D9 127.6 mm to (115.4, 100.6), turned to 93 degrees
- moved D10 116.2 mm to (133.1, 67.1), turned to 90 degrees
- moved D20 116.0 mm to (163.6, 125.3), turned to 87 degrees
- moved D11 110.5 mm to (133.3, 83.0), turned to 90 degrees
- moved D13 100.9 mm to (154.4, 68.2), turned to 87 degrees
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
Commit message: basic routing
Parts:
- added H1: oled_cover_1, kbd:M2_Hole_TH, F.Cu at (193.2, 115.0)
- added H2: oled_cover_2, kbd:M2_Hole_TH, F.Cu at (205.2, 120.7)
- added REF**: M2_Hole_TH_Outside, kbd:M2_Hole_TH_Outside, F.Cu at (152.2, 114.9)
- added REF**: M2_Hole_TH_Outside, kbd:M2_Hole_TH_Outside, F.Cu at (114.5, 97.5)
- added REF**: M2_Hole_TH_Outside, kbd:M2_Hole_TH_Outside, F.Cu at (153.3, 79.2)
- added REF**: M2_Hole_TH_Outside, kbd:M2_Hole_TH_Outside, F.Cu at (94.4, 105.3)
- added REF**: M2_Hole_TH_Outside, kbd:M2_Hole_TH_Outside, F.Cu at (152.8, 96.5)
- added REF**: M2_Hole_TH_Outside, kbd:M2_Hole_TH_Outside, F.Cu at (199.2, 117.5)
- added REF**: M2_Hole_TH_Outside, kbd:M2_Hole_TH_Outside, F.Cu at (119.1, 117.3)
- added REF**: M2_Hole_TH_Outside, kbd:M2_Hole_TH_Outside, F.Cu at (90.3, 88.8)
- added REF**: M2_Hole_TH_Outside, kbd:M2_Hole_TH_Outside, F.Cu at (111.0, 80.1)
- moved D9 21.1 mm to (130.6, 115.2), turned to 3 degrees
- moved D15 21.0 mm to (169.2, 116.0), turned to -3 degrees
- moved D3 9.97 mm to (86.0, 108.4), turned to 15 degrees
- moved D2 9.56 mm to (81.5, 91.8), turned to 15 degrees
- moved D19 4.40 mm to (134.6, 128.7)
- moved D21 4.35 mm to (186.7, 132.9)
- moved D20 4.30 mm to (163.6, 129.7)
- moved D14 3.27 mm to (154.4, 86.5)
- moved D8 2.48 mm to (114.9, 85.8)
- moved D7 1.12 mm to (112.2, 71.7)
- moved D5 1.09 mm to (110.8, 89.3)
- moved D4 1.05 mm to (107.1, 73.2)
- moved D1 0.95 mm to (88.0, 77.2)
- moved D6 0.79 mm to (113.2, 105.7)
- moved D12 0.22 mm to (133.9, 100.0)
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Connections:
- U1 pad 1: LED -> col5
- U1 pad 10: home -> col1
- U1 pad 11: bottom -> col0
- U1 pad 13: col0 -> unconnected-(U1-Pad13)
- U1 pad 14: col1 -> unconnected-(U1-Pad14)
- U1 pad 15: col2 -> unconnected-(U1-Pad15)
- U1 pad 16: col3 -> unconnected-(U1-Pad16)
- U1 pad 17: col4 -> unconnected-(U1-Pad17)
- U1 pad 18: col5 -> bottom
- U1 pad 19: unconnected-(U1-Pad19) -> home
- U1 pad 20: unconnected-(U1-Pad20) -> top
- U1 pad 7: unconnected-(U1-Pad7) -> col4
- U1 pad 8: buzzer -> col3
- U1 pad 9: top -> col2
Routing:
- net col2: track 0.00 -> 197.0 mm, vias 0 -> 5
- net col0: track 0.00 -> 196.2 mm, vias 0 -> 4
- net col3: track 0.00 -> 183.1 mm, vias 0 -> 5
- net col4: track 0.00 -> 167.3 mm, vias 0 -> 5
- net col1: track 0.00 -> 166.8 mm, vias 0 -> 4
- net col5: track 0.00 -> 162.8 mm, vias 0 -> 4
- net bottom: track 0.00 -> 157.0 mm
- net home: track 0.00 -> 122.0 mm
- net top: track 0.00 -> 118.0 mm
- net GND: track 0.00 -> 92.9 mm, vias 0 -> 3
- net thumb: track 0.00 -> 88.6 mm
- net data: track 0.00 -> 46.1 mm, vias 0 -> 2
- net reset: track 0.00 -> 41.6 mm, vias 0 -> 3
- net Net-(D3-Pad1): track 0.00 -> 27.8 mm, vias 0 -> 1
- net Net-(D2-Pad1): track 0.00 -> 27.8 mm, vias 0 -> 1
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