File: askew-kbd/askew-kbd.kicad_pcb (KiCad board)
At the start: 2 copper layers, 145.2 x 92.1 mm, 68 parts, among them J1 OLED, J2 MJ-4PP-9, SW1 SW_PUSH, SW10 SW_PUSH, SW11 SW_PUSH, SW12 SW_PUSH, SW13 SW_PUSH, SW14 SW_PUSH, SW15 SW_PUSH, SW16 SW_PUSH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

Commit message: routing
Parts:
- removed JP9: , kbd:JPC2
- moved D22 5.51 mm to (197.2, 126.5)
- moved J2 3.06 mm to (209.8, 112.2)
- moved RSW1 1.61 mm to (193.4, 107.4)
- moved JP4 1.15 mm to (197.1, 99.7), turned to -93 degrees
- moved JP8 1.15 mm to (197.1, 99.7), turned to -93 degrees
- moved JP1 0.97 mm to (202.8, 100.0), turned to -93 degrees
- moved JP5 0.97 mm to (202.8, 100.0), turned to -93 degrees
- moved D7 0.85 mm to (112.1, 72.5)
- moved D4 0.67 mm to (107.4, 73.8)
- moved JP3 0.41 mm to (199.0, 99.8)
- moved JP7 0.41 mm to (199.0, 99.8)
- moved JP2 0.27 mm to (200.9, 99.9)
- moved JP6 0.27 mm to (200.9, 99.9)
- moved D8 0.10 mm to (114.9, 85.7)
- moved D5 0.10 mm to (110.8, 89.4)
Connections:
- J2 pad C: Net-(J2-PadC) -> data
Routing:
- net GND: track 92.9 -> 23.4 mm, vias 3 -> 4
- net top: track 118.0 -> 164.8 mm, vias 0 -> 1
- net bottom: track 157.0 -> 203.1 mm, vias 0 -> 3
- net col0: track 196.2 -> 241.4 mm, vias 4 -> 5
- net col1: track 166.8 -> 210.4 mm, vias 4 -> 5
- net col2: track 197.0 -> 234.7 mm, vias 5 -> 6
- net thumb: track 88.6 -> 126.1 mm, vias 0 -> 1
- net VCC: track 16.2 -> 52.7 mm, vias 1 -> 3
- net home: track 122.0 -> 157.2 mm, vias 0 -> 1
- net col3: track 183.1 -> 216.6 mm, vias 5 -> 6
- net SCL: track 3.59 -> 33.0 mm, vias 1 -> 3
- net col5: track 162.8 -> 191.4 mm, vias 4 -> 5
- net SDA: track 11.1 -> 38.3 mm, vias 1 -> 3
- net col4: track 167.3 -> 186.3 mm, vias 5 -> 6
- net Net-(J2-PadC): track 14.7 -> 0.00 mm
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- added copper zone on B.Cu, net GND
- added copper zone on F.Cu, net GND

Commit message: routing finished
Parts:
- moved J2 0.11 mm to (209.7, 112.2)
Routing:
- net unconnected-(U1-Pad13): track 0.00 -> 13.2 mm, vias 0 -> 1
- net unconnected-(U1-Pad14): track 0.00 -> 11.5 mm, vias 0 -> 1
- net unconnected-(U1-Pad16): track 0.00 -> 11.1 mm, vias 0 -> 1
- net unconnected-(U1-Pad24): track 0.00 -> 10.8 mm, vias 0 -> 1
- net unconnected-(U1-Pad17): track 0.00 -> 10.6 mm, vias 0 -> 1
- net unconnected-(U1-Pad15): track 0.00 -> 10.1 mm, vias 0 -> 1
- net top: track 164.8 -> 160.3 mm
- net col1: track 210.4 -> 213.8 mm
- net reset: track 45.4 -> 42.7 mm
- net col0: track 241.4 -> 243.9 mm
- net col4: track 186.3 -> 184.5 mm
- net SDA: track 38.3 -> 39.9 mm
- net Net-(D12-Pad1): track 24.7 -> 23.1 mm
- net col2: track 234.7 -> 236.2 mm
- net bottom: track 203.1 -> 201.7 mm
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Other:
- board text added: "askew-kbd v1 pcb by bncpr"

Commit message: plates
Parts:
- moved J2 2.61 mm to (209.9, 109.7)
Routing:
- net GND: track 24.4 -> 32.6 mm
- net data: track 53.4 -> 50.7 mm
- net VCC: track 51.4 -> 48.9 mm
Changed lines of the file:
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@@
   )
   (footprint "kbd:MJ-4PP-9" (layer "F.Cu")
-    (at 209.65 112.25 -93)
+    (at 209.9 109.65 -93)
     (property "Sheetfile" "askew-kbd.kicad_sch")
     (property "Sheetname" "")
@@
   (via (at 195.646221 99.2) (size 0.8) (drill 0.4) (layers "F.Cu" "B.Cu") (net 33))
   (segment (start 197.125882 99.2) (end 197.126188 99.200306) (width 0.25) (layer "B.Cu") (net 33))
+  (segment (start 198.097854 107.063537) (end 198.097854 109.381956) (width 0.25) (layer "B.Cu") (net 33))
   (segment (start 204.295185 73.9) (end 205.205367 72.989818) (width 0.25) (layer "B.Cu") (net 33))
   (segment (start 196.28275 75.02119) (end 196.28275 77.424776) (width 0.25) (layer "B.Cu") (net 33))
-  (segment (start 198.076077 111.803733) (end 197.897854 111.981956) (width 0.25) (layer "B.Cu") (net 33))
+  (segment (start 206.494617 105.943967) (end 206.494617 111.574413) (width 0.25) (layer "B.Cu") (net 33))
   (segment (start 205.205367 72.989818) (end 206.054456 72.989818) (width 0.25) (layer "B.Cu") (net 33))
   (segment (start 196.28275 77.424776) (end 196.149817 77.557709) (width 0.25) (layer "B.Cu") (net 33))
   (segment (start 197.85 73.9) (end 197.40394 73.9) (width 0.25) (layer "B.Cu") (net 33))
-  (segment (start 197.897854 111.981956) (end 197.847854 111.981956) (width 0.25) (layer "B.Cu") (net 33))
-  (segment (start 206.294617 114.174413) (end 206.244617 114.174413) (width 0.25) (layer "B.Cu") (net 33))
+  (segment (start 198.226077 106.935314) (end 198.097854 107.063537) (width 0.25) (layer "B.Cu") (net 33))
   (segment (start 195.646221 99.2) (end 197.125882 99.2) (width 0.25) (layer "B.Cu") (net 33))
   (segment (start 197.40394 73.9) (end 196.28275 75.02119) (width 0.25) (layer "B.Cu") (net 33))
+  (segment (start 206.806016 105.632568) (end 206.494617 105.943967) (width 0.25) (layer "B.Cu") (net 33))
   (segment (start 197.073812 101.026188) (end 196.2494 101.8506) (width 0.25) (layer "F.Cu") (net 34))
   (segment (start 197.073812 100.199694) (end 197.073812 101.026188) (width 0.25) (layer "F.Cu") (net 34))
@@
   (via (at 200.8245 77.9) (size 0.8) (drill 0.4) (layers "F.Cu" "B.Cu") (net 38))
   (segment (start 200.15 92.313833) (end 199.300497 93.163336) (width 0.25) (layer "B.Cu") (net 38))
-  (segment (start 200.186648 112.436648) (end 200.2 112.45) (width 0.25) (layer "B.Cu") (net 38))
-  (segment (start 199.026188 99.300306) (end 199.598472 99.300306) (width 0.25) (layer "B.Cu") (net 38))
-  (segment (start 200.186648 108.487255) (end 200.186648 112.436648) (width 0.25) (layer "B.Cu") (net 38))
+  (segment (start 199.65 105.100607) (end 199.815609 105.266216) (width 0.25) (layer "B.Cu") (net 38))
+  (segment (start 200.436648 105.887255) (end 200.436648 109.836648) (width 0.25) (layer "B.Cu") (net 38))
   (segment (start 199.300497 93.163336) (end 199.300497 96.6) (width 0.25) (layer "B.Cu") (net 38))
-  (segment (start 199.876645 99.578479) (end 199.876645 100.744121) (width 0.25) (layer "B.Cu") (net 38))
-  (segment (start 200.2 112.862272) (end 199.25421 113.808062) (width 0.25) (layer "B.Cu") (net 38))
+  (segment (start 199.598472 99.300306) (end 199.876645 99.578479) (width 0.25) (layer "B.Cu") (net 38))
   (segment (start 204.85 77.95) (end 204.962856 78.062856) (width 0.25) (layer "B.Cu") (net 38))
-  (segment (start 199.65 100.970766) (end 199.65 107.781825) (width 0.25) (layer "B.Cu") (net 38))
   (segment (start 200.5495 78.386701) (end 200.15 78.786201) (width 0.25) (layer "B.Cu") (net 38))
+  (segment (start 199.876645 99.578479) (end 199.876645 100.744121) (width 0.25) (layer "B.Cu") (net 38))
+  (segment (start 200.45 109.85) (end 200.45 110.262272) (width 0.25) (layer "B.Cu") (net 38))
   (segment (start 199.026188 96.874309) (end 199.300497 96.6) (width 0.25) (layer "B.Cu") (net 38))
-  (segment (start 199.65 107.781825) (end 199.565609 107.866216) (width 0.25) (layer "B.Cu") (net 38))
-  (segment (start 199.876645 100.744121) (end 199.65 100.970766) (width 0.25) (layer "B.Cu") (net 38))
   (segment (start 200.8245 77.9) (end 200.5495 78.175) (width 0.25) (layer "B.Cu") (net 38))
-  (segment (start 200.2 112.45) (end 200.2 112.862272) (width 0.25) (layer "B.Cu") (net 38))
   (segment (start 200.15 78.786201) (end 200.15 92.313833) (width 0.25) (layer "B.Cu") (net 38))
-  (segment (start 199.598472 99.300306) (end 199.876645 99.578479) (width 0.25) (layer "B.Cu") (net 38))
+  (segment (start 199.026188 99.300306) (end 199.598472 99.300306) (width 0.25) (layer "B.Cu") (net 38))
+  (segment (start 199.65 100.970766) (end 199.65 105.100607) (width 0.25) (layer "B.Cu") (net 38))
+  (segment (start 200.45 110.262272) (end 199.50421 111.208062) (width 0.25) (layer "B.Cu") (net 38))
   (segment (start 200.5495 78.175) (end 200.5495 78.386701) (width 0.25) (layer "B.Cu") (net 38))
   (segment (start 204.962856 78.062856) (end 205.788589 78.062856) (width 0.25) (layer "B.Cu") (net 38))
   (segment (start 199.026188 99.300306) (end 199.026188 96.874309) (width 0.25) (layer "B.Cu") (net 38))
-  (segment (start 199.565609 107.866216) (end 200.186648 108.487255) (width 0.25) (layer "B.Cu") (net 38))
+  (segment (start 199.876645 100.744121) (end 199.65 100.970766) (width 0.25) (layer "B.Cu") (net 38))
+  (segment (start 200.436648 109.836648) (end 200.45 109.85) (width 0.25) (layer "B.Cu") (net 38))
+  (segment (start 199.815609 105.266216) (end 200.436648 105.887255) (width 0.25) (layer "B.Cu") (net 38))
   (segment (start 201.138299 83.386201) (end 201.138299 83.3) (width 0.25) (layer "F.Cu") (net 39))
   (segment (start 200.8745 83.65) (end 201.2245 83.3) (width 0.25) (layer "F.Cu") (net 39))
@@
   (segment (start 200.75 97.203406) (end 200.75 97.85) (width 0.25) (layer "B.Cu") (net 40))
   (segment (start 202.95 72.7) (end 205.764638 72.7) (width 0.25) (layer "F.Cu") (net 41))
-  (segment (start 202.297426 96.646408) (end 202.297426 97.736432) (width 0.25) (layer "F.Cu") (net 41))
-  (segment (start 203.484387 98.837831) (end 203.729021 99.082465) (width 0.25) (layer "F.Cu") (net 41))
-  (segment (start 203.398825 98.837831) (end 203.484387 98.837831) (width 0.25) (layer "F.Cu") (net 41))
+  (segment (start 203.729021 99.082465) (end 203.729021 99.929021) (width 0.25) (layer "F.Cu") (net 41))
   (segment (start 203.729021 99.929021) (end 205.05 101.25) (width 0.25) (layer "F.Cu") (net 41))
   (segment (start 202.297426 97.736432) (end 203.398825 98.837831) (width 0.25) (layer "F.Cu") (net 41))
-  (segment (start 205.05 101.25) (end 205.05 106.585687) (width 0.25) (layer "F.Cu") (net 41))
+  (segment (start 205.05 104.235687) (end 203.810127 105.47556) (width 0.25) (layer "F.Cu") (net 41))
   (segment (start 205.764638 72.7) (end 206.054456 72.989818) (width 0.25) (layer "F.Cu") (net 41))
-  (segment (start 205.05 106.585687) (end 203.560127 108.07556) (width 0.25) (layer "F.Cu") (net 41))
-  (segment (start 203.729021 99.082465) (end 203.729021 99.929021) (width 0.25) (layer "F.Cu") (net 41))
+  (segment (start 202.297426 96.646408) (end 202.297426 97.736432) (width 0.25) (layer "F.Cu") (net 41))
+  (segment (start 203.484387 98.837831) (end 203.729021 99.082465) (width 0.25) (layer "F.Cu") (net 41))
+  (segment (start 203.398825 98.837831) (end 203.484387 98.837831) (width 0.25) (layer "F.Cu") (net 41))
+  (segment (start 205.05 101.25) (end 205.05 104.235687) (width 0.25) (layer "F.Cu") (net 41))
   (via (at 202.297426 96.646408) (size 0.8) (drill 0.4) (layers "F.Cu" "B.Cu") (net 41))
   (via (at 202.95 72.7) (size 0.8) (drill 0.4) (layers "F.Cu" "B.Cu") (net 41))
@@
   (segment (start 202.95 72.7) (end 196.631012 72.7) (width 0.25) (layer "B.Cu") (net 41))
   (segment (start 202.575805 91.797216) (end 202.297426 92.075595) (width 0.25) (layer "B.Cu") (net 41))
-  (segment (start 203.248728 114.017405) (end 203.248728 108.386959) (width 0.25) (layer "B.Cu") (net 41))
+  (segment (start 203.498728 105.786959) (end 203.810127 105.47556) (width 0.25) (layer "B.Cu") (net 41))
   (segment (start 203.0005 72.7505) (end 203.0005 79.550305) (width 0.25) (layer "B.Cu") (net 41))
   (segment (start 203.0005 79.550305) (end 202.575805 79.975) (width 0.25) (layer "B.Cu") (net 41))
@@
   (segment (start 196.631012 72.7) (end 196.415683 72.484671) (width 0.25) (layer "B.Cu") (net 41))
   (segment (start 202.95 72.7) (end 203.0005 72.7505) (width 0.25) (layer "B.Cu") (net 41))
-  (segment (start 203.248728 108.386959) (end 203.560127 108.07556) (width 0.25) (layer "B.Cu") (net 41))
+  (segment (start 203.498728 111.417405) (end 203.498728 105.786959) (width 0.25) (layer "B.Cu") (net 41))
   (segment (start 194.624546 103.15) (end 193.620092 104.154454) (width 0.25) (layer "F.Cu") (net 42))
   (segment (start 200.111368 75.4) (end 204.35 75.4) (width 0.25) (layer "F.Cu") (net 42))

Commit message: v1
Parts:
- moved REF** 3.85 mm to (198.7, 121.3)
- moved H2 2.07 mm to (205.8, 122.7)
- moved H1 0.83 mm to (192.8, 115.8)
- moved RSW1 0.36 mm to (193.1, 107.5)
Routing:
- net reset: track 42.7 -> 45.9 mm
- net data: track 50.7 -> 53.7 mm
- net VCC: track 48.9 -> 51.1 mm
- net SDA: track 39.9 -> 41.6 mm
- net GND: track 32.6 -> 34.2 mm
- net col5: track 192.6 -> 194.1 mm
- net col1: track 213.8 -> 214.9 mm
- net unconnected-(U1-Pad15): track 10.1 -> 11.1 mm
- net home: track 157.7 -> 158.3 mm
- net unconnected-(U1-Pad16): track 11.1 -> 11.7 mm
- net col4: track 184.5 -> 185.1 mm
