File: askew-kbd/askew-kbd.kicad_sch (KiCad schematic)
At the start: 56 parts, among them J1 OLED, J2 MJ-4PP-9, SW1 SW_PUSH, SW10 SW_PUSH, SW11 SW_PUSH, SW12 SW_PUSH, SW13 SW_PUSH, SW14 SW_PUSH, SW15 SW_PUSH, SW16 SW_PUSH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

Commit message: plates
Connections:
- no-connect marks 0 -> 6
Changed lines of the file:
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@@
   (junction (at 142.24 37.465) (diameter 0) (color 0 0 0 0)
   )
+  (no_connect (at 91.44 74.93))
+  (no_connect (at 91.44 67.31))
+  (no_connect (at 91.44 46.99))
+  (no_connect (at 91.44 72.39))
+  (no_connect (at 91.44 69.85))
+  (no_connect (at 91.44 64.77))
   (wire (pts (xy 229.235 49.53) (xy 251.46 49.53))
     (stroke (width 0) (type default) (color 0 0 0 0))

Commit message: v1
Changed lines of the file:
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@@
+    (stroke (width 0) (type default) (color 0 0 0 0))
+  )
+  (wire (pts (xy 247.015 117.475) (xy 247.015 120.65))
+    (stroke (width 0) (type default) (color 0 0 0 0))
+  )
+  (wire (pts (xy 193.675 121.285) (xy 206.375 121.285))
+    (stroke (width 0) (type default) (color 0 0 0 0))
+  )
+  (wire (pts (xy 193.675 98.425) (xy 193.675 99.695))
+    (stroke (width 0) (type default) (color 0 0 0 0))
+  )
+  (wire (pts (xy 241.3 118.745) (xy 241.3 123.19))
+    (stroke (width 0) (type default) (color 0 0 0 0))
+  )
+  (wire (pts (xy 192.405 125.095) (xy 206.375 125.095))
+    (stroke (width 0) (type default) (color 0 0 0 0))
+  )
+  (wire (pts (xy 135.89 37.465) (xy 142.24 37.465))
+    (stroke (width 0) (type default) (color 0 0 0 0))
+  )
+  (wire (pts (xy 185.42 61.595) (xy 207.01 61.595))
+    (stroke (width 0) (type default) (color 0 0 0 0))
+  )
+  (wire (pts (xy 211.455 125.095) (xy 215.265 125.095))
+    (stroke (width 0) (type default) (color 0 0 0 0))
+  )
+  (wire (pts (xy 135.255 49.53) (xy 142.24 49.53))
+    (stroke (width 0) (type default) (color 0 0 0 0))
+  )
+  (wire (pts (xy 236.22 53.975) (xy 236.22 66.04))
+    (stroke (width 0) (type default) (color 0 0 0 0))
+  )
+  (wire (pts (xy 53.34 52.07) (xy 55.88 52.07))
+    (stroke (width 0) (type default) (color 0 0 0 0))
+  )
+  (wire (pts (xy 193.675 99.695) (xy 193.675 121.285))
+    (stroke (width 0) (type default) (color 0 0 0 0))
+  )
+  (wire (pts (xy 127 29.845) (xy 127 41.91))
+    (stroke (width 0) (type default) (color 0 0 0 0))
+  )
+  (wire (pts (xy 192.405 103.505) (xy 192.405 125.095))
+    (stroke (width 0) (type default) (color 0 0 0 0))
+  )
+  (wire (pts (xy 229.235 73.66) (xy 251.46 73.66))
+    (stroke (width 0) (type default) (color 0 0 0 0))
+  )
+  (wire (pts (xy 213.995 41.91) (xy 213.995 53.975))
+    (stroke (width 0) (type default) (color 0 0 0 0))
+  )
+  (wire (pts (xy 191.77 29.845) (xy 191.77 41.91))
+    (stroke (width 0) (type default) (color 0 0 0 0))
+  )
+  (wire (pts (xy 211.455 95.885) (xy 215.265 95.885))
+    (stroke (width 0) (type default) (color 0 0 0 0))
+  )
+  (wire (pts (xy 229.235 61.595) (xy 251.46 61.595))
+    (stroke (width 0) (type default) (color 0 0 0 0))
+  )
+  (wire (pts (xy 191.135 107.315) (xy 191.135 128.905))
+    (stroke (width 0) (type default) (color 0 0 0 0))
+  )
+  (wire (pts (xy 164.465 49.53) (xy 185.42 49.53))
+    (stroke (width 0) (type default) (color 0 0 0 0))
+  )
+  (wire (pts (xy 213.995 53.975) (xy 213.995 66.04))
+    (stroke (width 0) (type default) (color 0 0 0 0))
+  )
+  (wire (pts (xy 241.3 114.935) (xy 239.395 114.935))
+    (stroke (width 0) (type default) (color 0 0 0 0))
+  )
+  (wire (pts (xy 206.375 107.315) (xy 191.135 107.315))
+    (stroke (width 0) (type default) (color 0 0 0 0))
+  )
+  (wire (pts (xy 211.455 99.695) (xy 215.265 99.695))
+    (stroke (width 0) (type default) (color 0 0 0 0))
+  )
+  (wire (pts (xy 213.995 29.845) (xy 213.995 41.91))
+    (stroke (width 0) (type default) (color 0 0 0 0))
+  )
+  (wire (pts (xy 142.24 49.53) (xy 164.465 49.53))
+    (stroke (width 0) (type default) (color 0 0 0 0))
+  )
+  (wire (pts (xy 191.135 128.905) (xy 206.375 128.905))
+    (stroke (width 0) (type default) (color 0 0 0 0))
+  )
+  (wire (pts (xy 211.455 128.905) (xy 215.265 128.905))
+    (stroke (width 0) (type default) (color 0 0 0 0))
+  )
+  (wire (pts (xy 170.18 29.845) (xy 170.18 41.91))
+    (stroke (width 0) (type default) (color 0 0 0 0))
+  )
+  (wire (pts (xy 247.015 116.205) (xy 247.015 114.3))
+    (stroke (width 0) (type default) (color 0 0 0 0))
+  )
+  (wire (pts (xy 185.42 73.66) (xy 207.01 73.66))
+    (stroke (width 0) (type default) (color 0 0 0 0))
+  )
+  (wire (pts (xy 191.77 53.975) (xy 191.77 66.04))
+    (stroke (width 0) (type default) (color 0 0 0 0))
+  )
+  (wire (pts (xy 142.24 37.465) (xy 164.465 37.465))
+    (stroke (width 0) (type default) (color 0 0 0 0))
+  )
+  (wire (pts (xy 149.225 29.845) (xy 149.225 41.91))
+    (stroke (width 0) (type default) (color 0 0 0 0))
+  )
+  (wire (pts (xy 127 41.91) (xy 127 53.975))
+    (stroke (width 0) (type default) (color 0 0 0 0))
+  )
+  (wire (pts (xy 207.01 73.66) (xy 229.235 73.66))
     (stroke (width 0) (type default) (color 0 0 0 0))
   )
@@
     (stroke (width 0) (type default) (color 0 0 0 0))
   )
-  (wire (pts (xy 193.675 121.285) (xy 206.375 121.285))
-    (stroke (width 0) (type default) (color 0 0 0 0))
-  )
-  (wire (pts (xy 193.675 98.425) (xy 193.675 99.695))
-    (stroke (width 0) (type default) (color 0 0 0 0))
-  )
-  (wire (pts (xy 241.3 118.745) (xy 241.3 123.19))
-    (stroke (width 0) (type default) (color 0 0 0 0))
-  )
-  (wire (pts (xy 192.405 125.095) (xy 206.375 125.095))
-    (stroke (width 0) (type default) (color 0 0 0 0))
-  )
-  (wire (pts (xy 135.89 37.465) (xy 142.24 37.465))
-    (stroke (width 0) (type default) (color 0 0 0 0))
-  )
-  (wire (pts (xy 185.42 61.595) (xy 207.01 61.595))
-    (stroke (width 0) (type default) (color 0 0 0 0))
-  )
-  (wire (pts (xy 211.455 125.095) (xy 215.265 125.095))
-    (stroke (width 0) (type default) (color 0 0 0 0))
-  )
-  (wire (pts (xy 135.255 49.53) (xy 142.24 49.53))
-    (stroke (width 0) (type default) (color 0 0 0 0))
-  )
-  (wire (pts (xy 236.22 53.975) (xy 236.22 66.04))
-    (stroke (width 0) (type default) (color 0 0 0 0))
-  )
-  (wire (pts (xy 53.34 52.07) (xy 55.88 52.07))
-    (stroke (width 0) (type default) (color 0 0 0 0))
-  )
-  (wire (pts (xy 193.675 99.695) (xy 193.675 121.285))
-    (stroke (width 0) (type default) (color 0 0 0 0))
-  )
-  (wire (pts (xy 127 29.845) (xy 127 41.91))
-    (stroke (width 0) (type default) (color 0 0 0 0))
-  )
-  (wire (pts (xy 192.405 103.505) (xy 192.405 125.095))
-    (stroke (width 0) (type default) (color 0 0 0 0))
-  )
-  (wire (pts (xy 229.235 73.66) (xy 251.46 73.66))
-    (stroke (width 0) (type default) (color 0 0 0 0))
-  )
-  (wire (pts (xy 213.995 41.91) (xy 213.995 53.975))
-    (stroke (width 0) (type default) (color 0 0 0 0))
-  )
-  (wire (pts (xy 191.77 29.845) (xy 191.77 41.91))
-    (stroke (width 0) (type default) (color 0 0 0 0))
-  )
-  (wire (pts (xy 211.455 95.885) (xy 215.265 95.885))
-    (stroke (width 0) (type default) (color 0 0 0 0))
-  )
-  (wire (pts (xy 229.235 61.595) (xy 251.46 61.595))
-    (stroke (width 0) (type default) (color 0 0 0 0))
-  )
-  (wire (pts (xy 191.135 107.315) (xy 191.135 128.905))
-    (stroke (width 0) (type default) (color 0 0 0 0))
-  )
-  (wire (pts (xy 164.465 49.53) (xy 185.42 49.53))
-    (stroke (width 0) (type default) (color 0 0 0 0))
-  )
-  (wire (pts (xy 213.995 53.975) (xy 213.995 66.04))
-    (stroke (width 0) (type default) (color 0 0 0 0))
-  )
-  (wire (pts (xy 241.3 114.935) (xy 239.395 114.935))
-    (stroke (width 0) (type default) (color 0 0 0 0))
-  )
-  (wire (pts (xy 206.375 107.315) (xy 191.135 107.315))
-    (stroke (width 0) (type default) (color 0 0 0 0))
-  )
-  (wire (pts (xy 211.455 99.695) (xy 215.265 99.695))
-    (stroke (width 0) (type default) (color 0 0 0 0))
-  )
-  (wire (pts (xy 213.995 29.845) (xy 213.995 41.91))
-    (stroke (width 0) (type default) (color 0 0 0 0))
-  )
-  (wire (pts (xy 142.24 49.53) (xy 164.465 49.53))
-    (stroke (width 0) (type default) (color 0 0 0 0))
-  )
-  (wire (pts (xy 191.135 128.905) (xy 206.375 128.905))
-    (stroke (width 0) (type default) (color 0 0 0 0))
-  )
-  (wire (pts (xy 211.455 128.905) (xy 215.265 128.905))
-    (stroke (width 0) (type default) (color 0 0 0 0))
-  )
-  (wire (pts (xy 170.18 29.845) (xy 170.18 41.91))
-    (stroke (width 0) (type default) (color 0 0 0 0))
-  )
-  (wire (pts (xy 247.015 116.205) (xy 247.015 114.3))
-    (stroke (width 0) (type default) (color 0 0 0 0))
-  )
-  (wire (pts (xy 185.42 73.66) (xy 207.01 73.66))
-    (stroke (width 0) (type default) (color 0 0 0 0))
-  )
-  (wire (pts (xy 191.77 53.975) (xy 191.77 66.04))
-    (stroke (width 0) (type default) (color 0 0 0 0))
-  )
-  (wire (pts (xy 142.24 37.465) (xy 164.465 37.465))
-    (stroke (width 0) (type default) (color 0 0 0 0))
-  )
-  (wire (pts (xy 149.225 29.845) (xy 149.225 41.91))
-    (stroke (width 0) (type default) (color 0 0 0 0))
-  )
-  (wire (pts (xy 127 41.91) (xy 127 53.975))
-    (stroke (width 0) (type default) (color 0 0 0 0))
-  )
-  (wire (pts (xy 207.01 73.66) (xy 229.235 73.66))
-    (stroke (width 0) (type default) (color 0 0 0 0))
-  )
   (wire (pts (xy 170.18 53.975) (xy 170.18 66.04))
     (stroke (width 0) (type default) (color 0 0 0 0))
@@
   )
   (wire (pts (xy 241.3 112.395) (xy 241.3 114.935))
-    (stroke (width 0) (type default) (color 0 0 0 0))
-  )
-  (wire (pts (xy 247.015 117.475) (xy 247.015 118.745))
     (stroke (width 0) (type default) (color 0 0 0 0))
   )
@@
     )
   )
-  (global_label "data" (shape input) (at 247.015 118.745 0) (fields_autoplaced)
+  (global_label "data" (shape input) (at 247.015 120.65 0) (fields_autoplaced)
     (effects (font (size 1.524 1.524)) (justify left))
-    (property "Intersheet References" "${INTERSHEET_REFS}" (id 0) (at 147.955 33.02 0)
-      (effects (font (size 1.27 1.27)) hide)
-    )
+    (property "Intersheet References" "${INTERSHEET_REFS}" (id 0) (at 147.955 34.925 0)
+      (effects (font (size 1.27 1.27)) hide)
+    )
