File: plates/bottom/bottom.kicad_pcb (KiCad board)
At the start: 2 copper layers, 145.2 x 92.1 mm, 9 parts

Commit message: v1
Parts:
- moved REF** 3.85 mm to (200.7, 116.6)
Changed lines of the file:
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@@
   (setup
     (pad_to_mask_clearance 0)
+    (aux_axis_origin 154.200497 110.199158)
+    (grid_origin 154.200497 110.199158)
     (pcbplotparams
-      (layerselection 0x00010fc_ffffffff)
+      (layerselection 0x00010f0_ffffffff)
       (disableapertmacros false)
-      (usegerberextensions false)
+      (usegerberextensions true)
       (usegerberattributes true)
       (usegerberadvancedattributes true)
-      (creategerberjobfile true)
+      (creategerberjobfile false)
       (svguseinch false)
       (svgprecision 6)
@@
       (viasonmask false)
       (mode 1)
-      (useauxorigin false)
+      (useauxorigin true)
       (hpglpennumber 1)
       (hpglpenspeed 20)
@@
       (plotinvisibletext false)
       (sketchpadsonfab false)
-      (subtractmaskfromsilk false)
+      (subtractmaskfromsilk true)
       (outputformat 1)
       (mirror false)
-      (drillshape 1)
+      (drillshape 0)
       (scaleselection 1)
-      (outputdirectory "")
+      (outputdirectory "./gerber")
     )
   )
@@
     (at 154.800497 91.749158)
     (attr through_hole)
-    (fp_text reference "REF**" (at 0 0.5) (layer "F.SilkS")
+    (fp_text reference "REF**" (at 0 0.5) (layer "F.SilkS") hide
       (effects (font (size 1 1) (thickness 0.15)))
     )
-    (fp_text value "M2_Hole_TH" (at 0 -0.5) (layer "F.Fab")
+    (fp_text value "M2_Hole_TH" (at 0 -0.5) (layer "F.Fab") hide
       (effects (font (size 1 1) (thickness 0.15)))
     )
@@
     (at 116.500497 92.849158)
     (attr through_hole)
-    (fp_text reference "REF**" (at 0 0.5) (layer "F.SilkS")
+    (fp_text reference "REF**" (at 0 0.5) (layer "F.SilkS") hide
       (effects (font (size 1 1) (thickness 0.15)))
     )
-    (fp_text value "M2_Hole_TH" (at 0 -0.5) (layer "F.Fab")
+    (fp_text value "M2_Hole_TH" (at 0 -0.5) (layer "F.Fab") hide
       (effects (font (size 1 1) (thickness 0.15)))
     )
@@
     (at 96.400497 100.649158)
     (attr through_hole)
-    (fp_text reference "REF**" (at 0 0.5) (layer "F.SilkS")
+    (fp_text reference "REF**" (at 0 0.5) (layer "F.SilkS") hide
       (effects (font (size 1 1) (thickness 0.15)))
     )
-    (fp_text value "M2_Hole_TH" (at 0 -0.5) (layer "F.Fab")
+    (fp_text value "M2_Hole_TH" (at 0 -0.5) (layer "F.Fab") hide
       (effects (font (size 1 1) (thickness 0.15)))
     )
@@
     (at 92.300497 84.149158)
     (attr through_hole)
-    (fp_text reference "REF**" (at 0 0.5) (layer "F.SilkS")
+    (fp_text reference "REF**" (at 0 0.5) (layer "F.SilkS") hide
       (effects (font (size 1 1) (thickness 0.15)))
     )
-    (fp_text value "M2_Hole_TH" (at 0 -0.5) (layer "F.Fab")
+    (fp_text value "M2_Hole_TH" (at 0 -0.5) (layer "F.Fab") hide
       (effects (font (size 1 1) (thickness 0.15)))
     )
@@
   )
   (footprint "kbd:M2_Hole_TH" locked (layer "F.Cu")
-    (at 201.250497 112.799158)
+    (at 200.650497 116.599158)
     (attr through_hole)
-    (fp_text reference "REF**" (at 0 0.5) (layer "F.SilkS")
+    (fp_text reference "REF**" (at 0 0.5) (layer "F.SilkS") hide
       (effects (font (size 1 1) (thickness 0.15)))
     )
-    (fp_text value "M2_Hole_TH" (at 0 -0.5) (layer "F.Fab")
+    (fp_text value "M2_Hole_TH" (at 0 -0.5) (layer "F.Fab") hide
       (effects (font (size 1 1) (thickness 0.15)))
     )
@@
     (at 113.000497 75.399158)
     (attr through_hole)
-    (fp_text reference "REF**" (at 0 0.5) (layer "F.SilkS")
+    (fp_text reference "REF**" (at 0 0.5) (layer "F.SilkS") hide
       (effects (font (size 1 1) (thickness 0.15)))
     )
-    (fp_text value "M2_Hole_TH" (at 0 -0.5) (layer "F.Fab")
+    (fp_text value "M2_Hole_TH" (at 0 -0.5) (layer "F.Fab") hide
       (effects (font (size 1 1) (thickness 0.15)))
     )
@@
     (at 154.200497 110.199158)
     (attr through_hole)
-    (fp_text reference "REF**" (at 0 0.5) (layer "F.SilkS")
+    (fp_text reference "REF**" (at 0 0.5) (layer "F.SilkS") hide
       (effects (font (size 1 1) (thickness 0.15)))
     )
-    (fp_text value "M2_Hole_TH" (at 0 -0.5) (layer "F.Fab")
+    (fp_text value "M2_Hole_TH" (at 0 -0.5) (layer "F.Fab") hide
       (effects (font (size 1 1) (thickness 0.15)))
     )
@@
     (at 155.300497 74.499158)
     (attr through_hole)
-    (fp_text reference "REF**" (at 0 0.5) (layer "F.SilkS")
+    (fp_text reference "REF**" (at 0 0.5) (layer "F.SilkS") hide
       (effects (font (size 1 1) (thickness 0.15)))
     )
-    (fp_text value "M2_Hole_TH" (at 0 -0.5) (layer "F.Fab")
+    (fp_text value "M2_Hole_TH" (at 0 -0.5) (layer "F.Fab") hide
       (effects (font (size 1 1) (thickness 0.15)))
     )
@@
     (at 121.100497 112.649158)
     (attr through_hole)
-    (fp_text reference "REF**" (at 0 0.5) (layer "F.SilkS")
+    (fp_text reference "REF**" (at 0 0.5) (layer "F.SilkS") hide
       (effects (font (size 1 1) (thickness 0.15)))
     )
-    (fp_text value "M2_Hole_TH" (at 0 -0.5) (layer "F.Fab")
+    (fp_text value "M2_Hole_TH" (at 0 -0.5) (layer "F.Fab") hide
       (effects (font (size 1 1) (thickness 0.15)))
     )
