File: plates/top/top.kicad_pcb (KiCad board)
At the start: 2 copper layers, 144.1 x 92.1 mm, 33 parts, among them SW1 SW_PUSH, SW10 SW_PUSH, SW11 SW_PUSH, SW12 SW_PUSH, SW13 SW_PUSH, SW14 SW_PUSH, SW15 SW_PUSH, SW16 SW_PUSH, SW17 SW_PUSH, SW18 SW_PUSH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

Commit message: v1
Parts:
- removed H2: oled_cover_2, kbd:M2_Hole_TH_Outside
- removed the REF** at (201.5, 107.6)
- added REF**: M2_Hole_TH_Outside, kbd:M2_Hole_TH_Outside, F.Cu at (208.1, 112.8)
- added REF**: M2_Hole_TH_Outside, kbd:M2_Hole_TH_Outside, F.Cu at (195.1, 105.9)
- H1: footprint kbd:M2_Hole_TH_Outside -> kbd:M2_Hole_TH
- moved H1 8.33 mm to (200.9, 111.4)
Other:
- outline, holes or cut-outs redrawn
Changed lines of the file:
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@@
   (setup
     (pad_to_mask_clearance 0)
+    (aux_axis_origin 154.450497 105.049158)
+    (grid_origin 154.450497 105.049158)
     (pcbplotparams
-      (layerselection 0x00010fc_ffffffff)
+      (layerselection 0x00010f0_ffffffff)
       (disableapertmacros false)
-      (usegerberextensions false)
+      (usegerberextensions true)
       (usegerberattributes true)
       (usegerberadvancedattributes true)
-      (creategerberjobfile true)
+      (creategerberjobfile false)
       (svguseinch false)
       (svgprecision 6)
@@
       (viasonmask false)
       (mode 1)
-      (useauxorigin false)
+      (useauxorigin true)
       (hpglpennumber 1)
       (hpglpenspeed 20)
@@
       (plotinvisibletext false)
       (sketchpadsonfab false)
-      (subtractmaskfromsilk false)
+      (subtractmaskfromsilk true)
       (outputformat 1)
       (mirror false)
-      (drillshape 1)
+      (drillshape 0)
       (scaleselection 1)
-      (outputdirectory "")
+      (outputdirectory "./gerber")
     )
   )
@@
     (fp_line (start 9.525 -9.525) (end -9.525 -9.525) (layer "F.Fab") (width 0.15))
   )
-  (footprint "kbd:M2_Hole_TH_Outside" locked (layer "F.Cu")
-    (at 207.400497 110.849158)
-    (property "Sheetfile" "askew-kbd.kicad_sch")
-    (property "Sheetname" "")
-    (attr through_hole)
-    (fp_text reference "H2" (at 0 0.5) (layer "F.SilkS")
-      (effects (font (size 1 1) (thickness 0.15)))
-    )
-    (fp_text value "oled_cover_2" (at 0 -0.5) (layer "F.Fab")
-      (effects (font (size 1 1) (thickness 0.15)))
-    )
-    (pad "" thru_hole circle locked (at 0 0) (size 5 5) (drill 4) (layers *.Cu *.Mask))
-  )
   (footprint "kbd:SW_Hole" locked (layer "F.Cu")
     (at 100.450497 69.449158 13)
@@
     (pad "" thru_hole circle locked (at 0 0) (size 4.2 4.2) (drill 2.3) (layers *.Cu *.Mask))
   )
-  (footprint "kbd:M2_Hole_TH_Outside" locked (layer "F.Cu")
-    (at 195.450497 105.149158)
-    (property "Sheetfile" "askew-kbd.kicad_sch")
-    (property "Sheetname" "")
-    (attr through_hole)
-    (fp_text reference "H1" (at 0 0.5) (layer "F.SilkS")
-      (effects (font (size 1 1) (thickness 0.15)))
-    )
-    (fp_text value "oled_cover_1" (at 0 -0.5) (layer "F.Fab")
-      (effects (font (size 1 1) (thickness 0.15)))
-    )
-    (pad "" thru_hole circle locked (at 0 0) (size 5 5) (drill 4) (layers *.Cu *.Mask))
-  )
   (footprint "kbd:SW_Hole" locked (layer "F.Cu")
     (at 108.150497 102.849158 13)
@@
     (pad "" thru_hole circle locked (at 0 0) (size 4.2 4.2) (drill 2.3) (layers *.Cu *.Mask))
   )
-  (footprint "kbd:M2_Hole_TH" locked (layer "F.Cu")
-    (at 201.500497 107.649158)
-    (attr through_hole)
-    (fp_text reference "REF**" (at 0 0.5) (layer "F.SilkS") hide
-      (effects (font (size 1 1) (thickness 0.15)))
-    )
-    (fp_text value "M2_Hole_TH" (at 0 -0.5) (layer "F.Fab") hide
-      (effects (font (size 1 1) (thickness 0.15)))
-    )
-    (pad "" thru_hole circle locked (at 0 0) (size 4.2 4.2) (drill 2.3) (layers *.Cu *.Mask))
+  (footprint "kbd:M2_Hole_TH_Outside" (layer "F.Cu")
+    (at 208.100497 112.799158)
+    (attr through_hole board_only)
+    (fp_text reference "REF**" (at 0 0.5) (layer "F.SilkS") hide
+      (effects (font (size 1 1) (thickness 0.15)))
+    )
+    (fp_text value "M2_Hole_TH_Outside" (at 0 -0.5) (layer "F.Fab") hide
+      (effects (font (size 1 1) (thickness 0.15)))
+    )
+    (pad "" thru_hole circle locked (at 0 0) (size 5 5) (drill 4) (layers F&B.Cu *.Mask))
+    (pad "" thru_hole circle locked (at 0 0) (size 5 5) (drill 4) (layers F&B.Cu *.Mask))
   )
   (footprint "kbd:SW_Hole" locked (layer "F.Cu")
@@
     (fp_line (start 9.525 9.525) (end 9.525 -9.525) (layer "F.Fab") (width 0.15))
   )
+  (footprint "kbd:M2_Hole_TH" (layer "F.Cu")
+    (at 200.900497 111.449158)
+    (property "Sheetfile" "askew-kbd.kicad_sch")
+    (property "Sheetname" "")
+    (attr through_hole board_only)
+    (fp_text reference "H1" (at 0 0.5) (layer "F.SilkS") hide
+      (effects (font (size 1 1) (thickness 0.15)))
+    )
+    (fp_text value "oled_cover_1" (at 0 -0.5) (layer "F.Fab") hide
+      (effects (font (size 1 1) (thickness 0.15)))
+    )
+    (pad "" thru_hole circle locked (at 0 0) (size 4.2 4.2) (drill 2.3) (layers F&B.Cu *.Mask))
+  )
   (footprint "kbd:SW_Hole" locked (layer "F.Cu")
     (at 85.56806 89.651748 15)
@@
     (fp_line (start -9.525 9.525) (end 9.525 9.525) (layer "F.Fab") (width 0.15))
     (fp_line (start 9.525 -9.525) (end -9.525 -9.525) (layer "F.Fab") (width 0.15))
+  )
+  (footprint "kbd:M2_Hole_TH_Outside" (layer "F.Cu")
+    (at 195.100497 105.899158)
+    (attr through_hole board_only)
+    (fp_text reference "REF**" (at 0 0.5) (layer "F.SilkS") hide
+      (effects (font (size 1 1) (thickness 0.15)))
+    )
+    (fp_text value "M2_Hole_TH_Outside" (at 0 -0.5) (layer "F.Fab") hide
+      (effects (font (size 1 1) (thickness 0.15)))
+    )
+    (pad "" thru_hole circle locked (at 0 0) (size 5 5) (drill 4) (layers F&B.Cu *.Mask))
+    (pad "" thru_hole circle locked (at 0 0) (size 5 5) (drill 4) (layers F&B.Cu *.Mask))
   )
   (footprint "kbd:SW_Hole" locked (layer "F.Cu")
@@
   (gr_arc (start 154.500497 50.699158) (mid 155.207604 50.992051) (end 155.500497 51.699158) (layer "Edge.Cuts") (width 0.1))
   (gr_arc (start 109.650497 112.099158) (mid 110.207569 112.212056) (end 110.500497 112.699158) (layer "Edge.Cuts") (width 0.1))
-  (gr_line (start 194.103604 54.5912) (end 191.75 99.85) (layer "Edge.Cuts") (width 0.1))
+  (gr_line (start 194.103604 54.5912) (end 191.700497 100.649158) (layer "Edge.Cuts") (width 0.1))
   (gr_line (start 139.750497 126.949158) (end 112.900497 129.249157) (layer "Edge.Cuts") (width 0.1))
   (gr_line (start 166.650497 128.299158) (end 139.750497 126.949158) (layer "Edge.Cuts") (width 0.1))
@@
   (gr_arc (start 112.900497 129.249157) (mid 112.166854 129.029218) (end 111.801229 128.356222) (layer "Edge.Cuts") (width 0.1))
   (gr_line (start 198.341812 142.66179) (end 183.600497 134.149158) (layer "Edge.Cuts") (width 0.1))
-  (gr_line (start 213.199999 111.6) (end 211.300497 116.149158) (layer "Edge.Cuts") (width 0.1))
+  (gr_line (start 212.849999 112.45) (end 211.300497 116.149158) (layer "Edge.Cuts") (width 0.1))
   (gr_arc (start 212.900497 117.599158) (mid 213.355339 118.202618) (end 213.249503 118.950843) (layer "Edge.Cuts") (width 0.1))
-  (gr_arc (start 212.75 110.250001) (mid 213.254593 110.831803) (end 213.199999 111.6) (layer "Edge.Cuts") (width 0.1))
+  (gr_arc (start 212.4 111.100001) (mid 212.904593 111.681803) (end 212.849999 112.45) (layer "Edge.Cuts") (width 0.1))
   (gr_line (start 114.351235 56.40093) (end 88.946186 62.347476) (layer "Edge.Cuts") (width 0.1))
   (gr_arc (start 87.400497 61.599158) (mid 88.121436 61.67775) (end 88.605354 62.217892) (layer "Edge.Cuts") (width 0.1))
@@
   (gr_line (start 83.750497 117.699158) (end 109.650497 112.099158) (layer "Edge.Cuts") (width 0.1))
   (gr_line (start 183.600497 134.149158) (end 166.650497 128.299158) (layer "Edge.Cuts") (width 0.1))
-  (gr_line (start 191.75 99.85) (end 212.75 110.250001) (layer "Edge.Cuts") (width 0.1))
+  (gr_line (start 191.700497 100.649158) (end 212.4 111.100001) (layer "Edge.Cuts") (width 0.1))
   (gr_line (start 111.801229 128.356222) (end 110.500497 112.699158) (layer "Edge.Cuts") (width 0.1))
   (gr_line (start 213.249503 118.950843) (end 199.750497 142.349158) (layer "Edge.Cuts") (width 0.1))
   (gr_arc (start 211.850497 117.099158) (mid 211.421264 116.713452) (end 211.300497 116.149158) (layer "Edge.Cuts") (width 0.1))
-  (gr_text "askew-kbd v1\npcb by bncpr" (at 184.346578 107.745294) (layer "B.SilkS")
+  (gr_text "askew-kbd v1\npcb by bncpr" (at 182.6 110.8 -19) (layer "B.Mask")
     (effects (font (size 1 1) (thickness 0.15)) (justify mirror))
   )
-  (gr_text "askew-kbd v1\npcb by bncpr" (at 184.350497 107.749158) (layer "F.SilkS")
+  (gr_text "askew-kbd v1\npcb by bncpr" (at 182.8 110.9 -19) (layer "F.Mask")
     (effects (font (size 1 1) (thickness 0.15)))
   )
+  (target plus (at 155.05 86.65) (size 5) (width 0.1) (layer "Edge.Cuts"))
   (zone (net 0) (net_name "") (layer "F.Cu") (hatch edge 0.508)
     (connect_pads (clearance 0))
